File: minimoog-filter.brd (EAGLE design)
At the start: 160 x 100 mm, 58 parts, among them IC1 TL072D, Q1 BC857CSMD, T1 BC847, T10 BC847, T11 BC847, T12 BC847, T13 BC847, T14 BC847, T15 BC847, T2 BC847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

Commit message: moving
Connections:
- net N$29: now also R20.1
